File: KiCAD/system-on-a-business-card/sd_card.kicad_sch (KiCad schematic)
At the start: 8 parts, among them J4 Micro_SD_Card

Commit message: #10: mintor tweaks in routing, removed fiducials from bom, added values to buzzer and sd-card slot
Parts:
- J4: value Micro_SD_Card -> TF-018B-H15
Changed lines of the file:
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@@
       (effects (font (size 1.27 1.27)))
     )
-    (property "Value" "Micro_SD_Card" (at 173.99 57.15 0)
+    (property "Value" "TF-018B-H15" (at 173.99 57.15 0)
       (effects (font (size 1.27 1.27)))
     )
